File: beaver.kicad_sch (KiCad schematic)
At the start: 56 parts, among them J1 Conn_01x04_Male, J2 USB_C_Receptacle_USB2.0, J3 NFC, J4 Conn_01x17, J5 Conn_01x17, SW1 RESET, SW2 USER P0.17, U1 nRF52840, U2 USBLC6-2SC6, U4 AZ1117-3.3, Y1 Crystal_GND24_Small, Y2 Crystal_Small

Commit message: final touches
Parts:
- added C8: 100n, Capacitor_SMD:C_0402_1005Metric, symbol Device:C_Small
- C5, C6, C7: value 1uF -> 100n
- D2: renamed from D5; value YELLOW P0.24 -> Y P0.10
- D3: renamed from D6; value GREEN P0.22 -> G P1.13
- D4: renamed from D7; value RED P0.20 -> R P1.15
- D5: renamed from D3; value POWER -> PWR
- L1: footprint Inductor_SMD:L_0805_2012Metric -> Inductor_SMD:L_0402_1005Metric
- renumbered AE2 to AE1, C15 to C1, C18 to C10, C16 to C11, C19 to C12, C20 to C13, C24 to C14, C1 to C15, C2 to C16, C21 to C17, C22 to C18, C25 to C19, C10 to C2, C26 to C20, C3 to C21, C8 to C22, C4 to C23, C23 to C24, C17 to C3, C11 to C4, C27 to C9, J4 to J1, J5 to J2, J2 to J4, J1 to J5, R15 to R10, R5 to R11, R14 to R12, R7 to R13, R17 to R2, R18 to R3, R19 to R4, R2 to R5, R3 to R6, R6 to R7, R13 to R8, R4 to R9, U4 to U1, U1 to U2, U2 to U3, Y2 to Y1, Y1 to Y2
Connections:
- net GNDREF: now also Y2.2, Y2.4, C8.2
- net VDD: now also C8.1
- net ANT_MATCHED: now reaches AE1.1 (A), C15.1, L1.1
- net ANT: now reaches C16.1, L1.2, U2.H23 (ANT)
- net SWDCLK: now reaches J5.2 (Pin_2), U2.AA24 (SWDCLK)
- net SWDIO: now reaches J5.3 (Pin_3), U2.AC24 (SWDIO)
Other:
- note added: "Stackup JLC08161H-7628 8.28 mil prepreg L1-L2"
- moved on the sheet: AE1, C13, C14, C15, C16, C5, C6, C7, C9

Commit message: pre-release preparations
Parts:
- added JP1: LDO EN, Connector_PinHeader_2.54mm:PinHeader_1x02_P2.54mm_Vertical, symbol Jumper:Jumper_2_Bridged
- Y2: footprint Crystal:Crystal_SMD_3225-4Pin_3.2x2.5mm -> Crystal:Crystal_SMD_2520-4Pin_2.5x2.0mm
Connections:
- net VBUS: now also R13.2
- net VDD: now also JP1.2 (B); no longer C20.1, R13.2, U1.2 (VO)
- new net: C20.1, JP1.1 (A), U1.2 (VO)
Changed lines of the file:
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@@
 	)
 	(junction
-		(at 194.31 99.06)
-		(diameter 0)
-		(color 0 0 0 0)
-	)
-	(junction
 		(at 24.13 119.38)
 		(diameter 0)
@@
 	)
 	(junction
+		(at 194.31 99.06)
+		(diameter 0)
+		(color 0 0 0 0)
+	)
+	(junction
 		(at 267.97 138.43)
 		(diameter 0)
@@
 	(wire
 		(pts
-			(xy 148.59 74.93) (xy 158.75 74.93)
+			(xy 194.31 99.06) (xy 198.12 99.06)
 		)
 		(stroke
@@
 	(wire
 		(pts
-			(xy 20.32 162.56) (xy 48.26 162.56)
+			(xy 148.59 74.93) (xy 158.75 74.93)
 		)
 		(stroke
@@
 	(wire
 		(pts
-			(xy 114.3 83.82) (xy 127 83.82)
+			(xy 20.32 162.56) (xy 48.26 162.56)
 		)
 		(stroke
@@
 	(wire
 		(pts
-			(xy 269.24 138.43) (xy 267.97 138.43)
+			(xy 114.3 83.82) (xy 127 83.82)
 		)
 		(stroke
@@
 	(wire
 		(pts
-			(xy 212.09 152.4) (xy 212.09 148.59)
+			(xy 269.24 138.43) (xy 267.97 138.43)
 		)
 		(stroke
@@
 	(wire
 		(pts
-			(xy 73.66 191.77) (xy 66.04 191.77)
+			(xy 212.09 152.4) (xy 212.09 148.59)
 		)
 		(stroke
@@
 	(wire
 		(pts
-			(xy 66.04 43.18) (xy 66.04 17.78)
+			(xy 73.66 191.77) (xy 66.04 191.77)
 		)
 		(stroke
@@
 	(wire
 		(pts
-			(xy 267.97 74.93) (xy 255.27 74.93)
+			(xy 66.04 43.18) (xy 66.04 17.78)
 		)
 		(stroke
@@
 	(wire
 		(pts
-			(xy 194.31 95.25) (xy 194.31 99.06)
+			(xy 267.97 74.93) (xy 255.27 74.93)
 		)
 		(stroke
@@
 	(wire
 		(pts
-			(xy 60.96 191.77) (xy 57.15 191.77)
+			(xy 60.96 191.77) (xy 52.07 191.77)
 		)
 		(stroke
@@
 	(wire
 		(pts
+			(xy 210.82 96.52) (xy 210.82 99.06)
+		)
+		(stroke
+			(width 0)
+			(type default)
+		)
+	)
+	(wire
+		(pts
 			(xy 129.54 20.32) (xy 139.7 20.32)
 		)
@@
 	(wire
 		(pts
-			(xy 57.15 191.77) (xy 57.15 189.23)
+			(xy 52.07 191.77) (xy 52.07 189.23)
 		)
 		(stroke
@@
 	(wire
 		(pts
+			(xy 210.82 99.06) (xy 208.28 99.06)
+		)
+		(stroke
+			(width 0)
+			(type default)
+		)
+	)
+	(wire
+		(pts
 			(xy 114.3 86.36) (xy 127 86.36)
 		)
@@
 			)
 		)
-		(property "Footprint" "Crystal:Crystal_SMD_3225-4Pin_3.2x2.5mm"
+		(property "Footprint" "Crystal:Crystal_SMD_2520-4Pin_2.5x2.0mm"
 			(at 38.1 114.3 0)
 			(effects
@@
 	)
 	(symbol
-		(lib_id "power:VDD")
-		(at 57.15 189.23 0)
-		(unit 1)
-		(exclude_from_sim no)
-		(in_bom yes)
-		(on_board yes)
-		(dnp no)
-		(property "Reference" "#PWR034"
-			(at 57.15 193.04 0)
-			(effects
-				(font
-					(size 1.27 1.27)
-				)
-				(hide yes)
-			)
-		)
-		(property "Value" "VDD"
-			(at 57.531 184.8358 0)
-			(effects
-				(font
-					(size 1.27 1.27)
-				)
-			)
-		)
-		(property "Footprint" ""
-			(at 57.15 189.23 0)
-			(effects
-				(font
-					(size 1.27 1.27)
-				)
-				(hide yes)
-			)
-		)
-		(property "Datasheet" ""
-			(at 57.15 189.23 0)
-			(effects
-				(font
-					(size 1.27 1.27)
-				)
-				(hide yes)
-			)
-		)
-		(property "Description" ""
-			(at 57.15 189.23 0)
-			(effects
-				(font
-					(size 1.27 1.27)
-				)
-				(hide yes)
-			)
-		)
-		(pin "1"
-		)
-		(instances
-			(project "beaver"
-				(path "/834ac438-0162-459a-8b70-ce62670b4c91"
-					(reference "#PWR034")
-					(unit 1)
-				)
-			)
-		)
-	)
-	(symbol
 		(lib_id "Device:C_Small")
 		(at 148.59 69.85 0)
@@
 	(symbol
 		(lib_id "power:VDD")
-		(at 194.31 95.25 0)
+		(at 210.82 96.52 0)
 		(unit 1)
 		(exclude_from_sim no)
@@
 		(dnp no)
 		(property "Reference" "#PWR019"
-			(at 194.31 99.06 0)
+			(at 210.82 100.33 0)
 			(effects
 				(font
@@
 		)
 		(property "Value" "VDD"
-			(at 194.691 90.8558 0)
+			(at 211.201 92.1258 0)
 			(effects
 				(font
@@
 		)
 		(property "Footprint" ""
-			(at 194.31 95.25 0)
+			(at 210.82 96.52 0)
 			(effects
 				(font
@@
 		)
 		(property "Datasheet" ""
-			(at 194.31 95.25 0)
+			(at 210.82 96.52 0)
 			(effects
 				(font
@@
 		)
 		(property "Description" ""
-			(at 194.31 95.25 0)
+			(at 210.82 96.52 0)
 			(effects
 				(font
@@
 	)
 	(symbol
+		(lib_id "power:VBUS")
+		(at 52.07 189.23 0)
+		(unit 1)
+		(exclude_from_sim no)
+		(in_bom yes)
+		(on_board yes)
+		(dnp no)
+		(property "Reference" "#PWR037"
+			(at 52.07 193.04 0)
+			(effects
+				(font
+					(size 1.27 1.27)
+				)
+				(hide yes)
+			)
+		)
+		(property "Value" "VBUS"
+			(at 52.451 184.8358 0)
+			(effects
+				(font
+					(size 1.27 1.27)
+				)
+			)
+		)
+		(property "Footprint" ""
+			(at 52.07 189.23 0)
+			(effects
+				(font
+					(size 1.27 1.27)
+				)
+				(hide yes)
+			)
+		)
+		(property "Datasheet" ""
+			(at 52.07 189.23 0)
+			(effects
+				(font
+					(size 1.27 1.27)
+				)
+				(hide yes)
+			)
+		)
+		(property "Description" ""
+			(at 52.07 189.23 0)
+			(effects
+				(font
+					(size 1.27 1.27)
+				)
+				(hide yes)
+			)
+		)
+		(pin "1"
+		)
+		(instances
+			(project "beaver"
+				(path "/834ac438-0162-459a-8b70-ce62670b4c91"
+					(reference "#PWR037")
+					(unit 1)
+				)
+			)
+		)
+	)
+	(symbol
 		(lib_id "Connector_Generic:Conn_01x17")
 		(at 240.03 67.31 0)
@@
 					(unit 1)
 				)
+			)
+		)
+	)
+	(symbol
+		(lib_id "Jumper:Jumper_2_Bridged")
+		(at 203.2 99.06 0)
+		(unit 1)
+		(exclude_from_sim yes)
+		(in_bom yes)
+		(on_board yes)
+		(dnp no)
+		(fields_autoplaced yes)
+		(property "Reference" "JP1"
+			(at 203.2 93.98 0)
+			(effects
+				(font
+					(size 1.27 1.27)
+				)
+			)
+		)
+		(property "Value" "LDO EN"
+			(at 203.2 96.52 0)
+			(effects
+				(font
+					(size 1.27 1.27)
+				)
+			)
+		)
+		(property "Footprint" "Connector_PinHeader_2.54mm:PinHeader_1x02_P2.54mm_Vertical"
+			(at 203.2 99.06 0)
+			(effects
+				(font
+					(size 1.27 1.27)
+				)
+				(hide yes)
+			)
+		)
+		(property "Datasheet" "~"
+			(at 203.2 99.06 0)
+			(effects
+				(font
+					(size 1.27 1.27)
+				)
+				(hide yes)
+			)
+		)
+		(property "Description" "Jumper, 2-pole, closed/bridged"
+			(at 203.2 99.06 0)
+			(effects
+				(font
+					(size 1.27 1.27)
+				)
+				(hide yes)
+			)
+		)
+		(pin "2"
+		)
+		(pin "1"
+		)
+		(instances
+			(project "beaver"
+				(path "/834ac438-0162-459a-8b70-ce62670b4c91"
+					(reference "JP1")
+					(unit 1)
+				)

Commit message: switch stackup for cost measures
Other:
- note added: "Stackup JLC08161H-2116 4.58 mil prepreg L1-L2"
- note removed: "Stackup JLC08161H-7628 8.28 mil prepreg L1-L2"
Changed lines of the file:
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@@
 		)
 	)
-	(text "Stackup JLC08161H-7628\n8.28 mil prepreg L1-L2"
+	(text "Stackup JLC08161H-2116\n4.58 mil prepreg L1-L2"
 		(exclude_from_sim no)
 		(at 251.714 153.67 0)

Commit message: switch to 6 layer stackup
Parts:
- D2: value Y P0.10 -> Y P1.13
- D3: value G P1.13 -> G P1.15
- D4: value R P1.15 -> R P0.2
Connections:
- net P0.2: now also D4.1 (K); no longer J1.6 (Pin_6)
- net P0.29: now also J1.4 (Pin_4); no longer J2.1 (Pin_1)
- net P0.3: now also R6.2; no longer R5.2
- net P0.30: now also R1.2; no longer R6.2
- net P0.31: now also J1.5 (Pin_5); no longer J1.4 (Pin_4)
- net P0.5: now also J1.6 (Pin_6); no longer J1.5 (Pin_5)
- net P1.10: now also J2.1 (Pin_1); no longer D2.1 (K)
- net P1.12: now also R5.2; no longer R1.2
- net P1.13: now also D2.1 (K); no longer D3.1 (K)
- net P1.15: now also D3.1 (K); no longer D4.1 (K)
- net RESET: now also C24.1, R8.2, SW2.1 (C); no longer C22.1, R7.2, SW1.1 (C)
- net USER_BUT: now also C22.1, R7.2, SW1.1 (C); no longer C24.1, R8.2, SW2.1 (C)
Other:
- note added: "Stackup JLC06061H-3313 3.91 mil prepreg L1-L2"
- note removed: "Stackup JLC08161H-2116 4.58 mil prepreg L1-L2"
Changed lines of the file:
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@@
 	(wire
 		(pts
+			(xy 262.89 43.18) (xy 262.89 36.83)
+		)
+		(stroke
+			(width 0)
+			(type default)
+		)
+	)
+	(wire
+		(pts
 			(xy 40.64 114.3) (xy 43.18 114.3)
 		)
@@
 	(wire
 		(pts
+			(xy 251.46 36.83) (xy 255.27 36.83)
+		)
+		(stroke
+			(width 0)
+			(type default)
+		)
+	)
+	(wire
+		(pts
 			(xy 86.36 27.94) (xy 86.36 34.29)
 		)
@@
 	(wire
 		(pts
+			(xy 270.51 41.91) (xy 270.51 36.83)
+		)
+		(stroke
+			(width 0)
+			(type default)
+		)
+	)
+	(wire
+		(pts
 			(xy 114.3 91.44) (xy 127 91.44)
 		)
@@
 		)
 	)
-	(text "Stackup JLC08161H-2116\n4.58 mil prepreg L1-L2"
+	(text "Stackup JLC06061H-3313\n3.91 mil prepreg L1-L2"
 		(exclude_from_sim no)
 		(at 251.714 153.67 0)
@@
 	)
 	(label "P0.3"
-		(at 232.41 25.4 180)
+		(at 232.41 30.48 180)
 		(fields_autoplaced yes)
 		(effects
@@
 	)
 	(label "P1.13"
-		(at 262.89 36.83 0)
+		(at 251.46 36.83 180)
 		(fields_autoplaced yes)
 		(effects
@@
 				(size 1.27 1.27)
 			)
-			(justify left bottom)
+			(justify right bottom)
 		)
 	)
 	(label "P0.5"
-		(at 220.98 57.15 180)
+		(at 220.98 59.69 180)
 		(fields_autoplaced yes)
 		(effects
@@
 	)
 	(label "P1.12"
-		(at 232.41 20.32 180)
+		(at 232.41 25.4 180)
 		(fields_autoplaced yes)
 		(effects
@@
 	)
 	(label "P0.2"
-		(at 220.98 59.69 180)
+		(at 270.51 41.91 0)
 		(fields_autoplaced yes)
 		(effects
@@
 				(size 1.27 1.27)
 			)
-			(justify right bottom)
+			(justify left bottom)
 		)
 	)
@@
 	)
 	(label "P0.30"
-		(at 232.41 30.48 180)
+		(at 232.41 20.32 180)
 		(fields_autoplaced yes)
 		(effects
@@
 	)
 	(label "USER_BUT"
-		(at 259.08 138.43 0)
+		(at 256.54 109.22 0)
 		(fields_autoplaced yes)
 		(effects
@@
 	)
 	(label "P0.31"
-		(at 220.98 54.61 180)
+		(at 220.98 57.15 180)
 		(fields_autoplaced yes)
 		(effects
@@
 	)
 	(label "P1.15"
-		(at 270.51 36.83 0)
+		(at 262.89 43.18 180)
 		(fields_autoplaced yes)
 		(effects
@@
 				(size 1.27 1.27)
 			)
-			(justify left bottom)
+			(justify right bottom)
 		)
 	)
 	(label "RESET"
-		(at 256.54 109.22 0)
+		(at 259.08 138.43 0)
 		(fields_autoplaced yes)
 		(effects
@@
 	)
 	(label "P0.29"
-		(at 267.97 87.63 0)
+		(at 220.98 54.61 180)
 		(fields_autoplaced yes)
 		(effects
@@
 				(size 1.27 1.27)
 			)
-			(justify left bottom)
+			(justify right bottom)
 		)
 	)
@@
 	)
 	(label "P1.10"
-		(at 255.27 36.83 0)
+		(at 267.97 87.63 0)
 		(fields_autoplaced yes)
 		(effects
@@
 			)
 		)
-		(property "Value" "R P1.15"
-			(at 273.5072 34.3408 90)
+		(property "Value" "R P0.2"
+			(at 270.51 39.116 90)
 			(effects
 				(font
@@
 			)
 		)
-		(property "Value" "G P1.13"
-			(at 260.096 40.132 90)
+		(property "Value" "G P1.15"
+			(at 256.54 40.132 90)
 			(effects
 				(font
@@
 			)
 		)
-		(property "Value" "Y P0.10"
-			(at 245.618 32.766 90)
+		(property "Value" "Y P1.13"
+			(at 244.856 33.782 90)
 			(effects
 				(font
